File: ANE21_PCB.kicad_pcb (KiCad board)
At the start: 4 copper layers, 74.6 x 66 mm, 60 parts, among them J13 1-2199119-5, J15 USB_OTG, J16 Conn_01x02, J2 Barrel_Jack, J3 USB-A-S-VT, J5 690-019-298-412, J6 Conn_02x07_Odd_Even, J7 2036150003 (USB-C_Connector), U1 74LVC1G07SE-7, U10 PUSB3FR4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

Commit message: definitief ingelverd
Parts:
- removed H1, H2, H3, H4, H5, H6, H7, H8: MountingHole, MountingHole:MountingHole_2.7mm_M2.5
Routing:
- removed copper zone on B.Cu, net GND
- removed copper zone on F.Cu, net GND
