File: ANE21_PCB_Gerbers/ANE21_PCB.kicad_pcb (KiCad board)
At the start: 4 copper layers, 59.6 x 61.6 mm, 58 parts, among them J1 1-2199119-5, J2 USB4105-GF-A, J3 USB-A-S-VT, J4 HDMI_A_1.4, J5 Conn_02x05_Odd_Even, J6 Conn_01x02, J8 Conn_02x06_Odd_Even, SW1 SW_Push, SW2 SW_Push, SW3 SW_Push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

Commit message: gerber files gemaakt
Parts:
- moved J6 0.62 mm to (115.6, 75.1)
Routing:
- net VBUS-PD: track 37.3 -> 36.7 mm
Changed lines of the file:
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@@
 	(footprint "1-2199119-5_Finley:TerminalBlock_PhoenixTerminalBlock_Phoenix_MKDS-1,5-2-5.08_1x02_P5.08mm_Horizontal_Edited"
 		(layer "B.Cu")
-		(at 116.2325 75.129163 -90)
+		(at 115.608483 75.129163 -90)
 		(property "Reference" "J6"
 			(at 0 0.5 90)
@@
 	)
 	(segment
-		(start 114.581663 81.02)
-		(end 118.5925 77.009163)
+		(start 112.47 81.02)
+		(end 113.957646 81.02)
 		(width 0.5)
 		(layer "B.Cu")
@@
 	)
 	(segment
-		(start 112.47 81.02)
-		(end 114.581663 81.02)
-		(width 0.5)
-		(layer "B.Cu")
-		(net 208)
-	)
-	(segment
 		(start 110.735 86.255)
 		(end 110.735 85.185)
@@
 		(width 0.5)
 		(layer "B.Cu")
+		(net 208)
+	)
+	(segment
+		(start 113.957646 81.02)
+		(end 117.968483 77.009163)
+		(width 0.5)
+		(layer "B.Cu")
